File: pcb/cbb-gpio/mk1-cbb.kicad_pcb (KiCad board)
At the start: 2 copper layers, 67.1 x 57.9 mm, 71 parts, among them J1 Conn_02x06_Odd_Even, J14 Screw_Terminal_01x08, J2 Screw_Terminal_01x04, J3 Screw_Terminal_01x06, J4 Screw_Terminal_01x06, Q1 AO3400A, Q10 AO3400A, Q2 AO3400A, Q3 AO3400A, Q4 AO3400A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

Commit message: add slim CBB
Other:
- board text added: "CocktailBerryBoard v0.5 07/2026"
- board text removed: "CocktailBerryBoard v0.4-lite 05/2025"
Changed lines of the file:
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@@
 		)
 	)
-	(gr_text "CocktailBerryBoard\nv0.4-lite\n05/2025"
+	(gr_text "CocktailBerryBoard\nv0.5\n07/2026"
 		(at 213.233 66.675 0)
 		(layer "B.SilkS")
@@
 	)
 	(gr_text "JLCJLCJLCJLC"
-		(at 188.214 97.79 0)
+		(at 213 70.5 0)
 		(layer "B.SilkS")
 		(effects
