File: pcb/cbb-gpio/mk1-cbb.kicad_pcb (KiCad board)
At the start: 2 copper layers, 67.1 x 57.9 mm, 71 parts, among them J1 Conn_02x06_Odd_Even, J14 Screw_Terminal_01x08, J2 Screw_Terminal_01x04, J3 Screw_Terminal_01x06, J4 Screw_Terminal_01x06, Q1 AO3400A, Q10 AO3400A, Q2 AO3400A, Q3 AO3400A, Q4 AO3400A, Q5 AO3400A, Q6 AO3400A, Q7 AO3400A, Q8 AO3400A, Q9 AO3400A

Commit message: Adjust board version numbering
Other:
- board text added: "CocktailBerryBoard v1.0 09/2026"
- board text removed: "CocktailBerryBoard v0.5 07/2026"
Changed lines of the file:
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@@
 		)
 	)
-	(gr_text "CocktailBerryBoard\nv0.5\n07/2026"
+	(gr_text "CocktailBerryBoard\nv1.0\n09/2026"
 		(at 213.233 66.675 0)
 		(layer "B.SilkS")
