File: pcb/cbb-slim/mk1-slim.kicad_sch (KiCad schematic)
At the start: 10 parts, among them J1 Screw_Terminal_01x08, J2 Screw_Terminal_01x04, J3 Conn_01x05, J5 Conn_01x05, J6 Screw_Terminal_01x08

Commit message: adjust mpn property spelling
Parts:
- F1: MPN (none) -> C22396288; mpn C22396288 -> (none)
- J2: MPN (none) -> C430624; mpn C430624 -> (none); now in the parts list
- J3, J5: MPN (none) -> C124379; mpn C124379 -> (none)
Changed lines of the file:
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@@
 			)
 		)
-		(property "mpn" "C22396288"
+		(property "MPN" "C22396288"
 			(at 111.76 99.06 90)
 			(effects
@@
 			)
 		)
-		(property "mpn" "C124379"
+		(property "MPN" "C124379"
 			(at 135.89 46.99 0)
 			(effects
@@
 		(unit 1)
 		(exclude_from_sim no)
-		(in_bom no)
+		(in_bom yes)
 		(on_board yes)
 		(dnp no)
@@
 			)
 		)
-		(property "mpn" "C430624"
+		(property "MPN" "C430624"
 			(at 119.38 91.44 90)
 			(effects
@@
 			)
 		)
-		(property "mpn" "C124379"
+		(property "MPN" "C124379"
 			(at 135.89 62.23 0)
 			(effects
