File: pcb/cbb-slim/mk1-slim.kicad_pcb (KiCad board)
At the start: 2 copper layers, 110.6 x 32.2 mm, 59 parts, among them J1 Screw_Terminal_01x08, J2 Screw_Terminal_01x04, J3 Conn_01x05, J5 Conn_01x05, J6 Screw_Terminal_01x08, Q1 AO3400A, Q10 AO3400A, Q2 AO3400A, Q3 AO3400A, Q6 AO3400A, Q7 AO3400A, Q8 AO3400A, Q9 AO3400A

Commit message: Adjust board version numbering
Other:
- board text added: "CocktailBerryBoard slim-v1.0 09/2026"
- board text removed: "CocktailBerryBoard slim-v0.3 07/2026"
Changed lines of the file:
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@@
 		(layer "Edge.Cuts")
 	)
-	(gr_text "CocktailBerryBoard\nslim-v0.3\n07/2026"
+	(gr_text "CocktailBerryBoard\nslim-v1.0\n09/2026"
 		(at 191.456823 62.668503 0)
 		(layer "B.SilkS")
