File: pcb/cbb-i2c/pump_control.kicad_sch (KiCad schematic)
At the start: 6 parts, among them Q5 AO3400A

Commit message: reduce brightness of channel indicator led
Parts:
- R16: value 220 -> 680; MPN C22962 -> C23228
Changed lines of the file:
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@@
 			)
 		)
-		(property "Value" "220"
+		(property "Value" "680"
 			(at 92.71 90.17 0)
 			(effects
@@
 			)
 		)
-		(property "MPN" "C22962"
+		(property "MPN" "C23228"
 			(at 99.06 88.9 90)
 			(effects
